File: HighSideSwitch.kicad_sch (KiCad schematic)
At the start: 24 parts, among them J1 Conn_02x02_Odd_Even, Q1 CSD18540Q5B, Q2 CSD18540Q5B, Q3 8050, U1 LM5060, U2 LM5050-1

Commit message: S
Parts:
- removed C1, C3, C4: 100n, Capacitor_SMD:C_0402_1005Metric, symbol Device:C_Small
- removed D1: VS-6ESU06, Package_TO_SOT_SMD:TO-277A, symbol Diode:VS-6ESU06
- removed D2: LED, LED_SMD:LED_0603_1608Metric, symbol Device:LED
- removed H1, H2: MountingHole_Pad, MountingHole:MountingHole_3.2mm_M3_Pad_Via, symbol Mechanical:MountingHole_Pad
- removed J1: Conn_02x02_Odd_Even, Connector_PinHeader_1.27mm:PinHeader_2x02_P1.27mm_Vertical_SMD, symbol Connector_Generic:Conn_02x02_Odd_Even
- removed Q1, Q2: CSD18540Q5B, Package_TO_SOT_SMD:TDSON-8-1, symbol Transistor_FET:CSD18540Q5B
- removed Q3: 8050, Package_TO_SOT_SMD:TSOT-23, symbol Device:Q_NPN_BEC
- removed R1: 9K, Resistor_SMD:R_0402_1005Metric, symbol Device:R_Small
- removed R10, R11, R8: 10K, Resistor_SMD:R_0402_1005Metric, symbol Device:R_Small
- removed R2, R9: 100, Resistor_SMD:R_0402_1005Metric, symbol Device:R_Small
- removed R3: 200K, Resistor_SMD:R_0402_1005Metric, symbol Device:R_Small
- removed R4: 100K, Resistor_SMD:R_0402_1005Metric, symbol Device:R_Small
- removed R5: 38.3K, Resistor_SMD:R_0402_1005Metric, symbol Device:R_Small
- removed R6: 14K, Resistor_SMD:R_0402_1005Metric, symbol Device:R_Small
- removed R7: 47K, Resistor_SMD:R_0402_1005Metric, symbol Device:R_Small
- removed U1: LM5060, Package_SO:MSOP-10_3x3mm_P0.5mm, symbol Power_Management:LM5060
- removed U2: LM5050-1, Package_TO_SOT_SMD:TSOT-23-6, symbol Power_Management:LM5050-1
- added C1, C3, C4: 100n, GENERAL_RCL_SMD:C0402(1005M), symbol Basic_passive_components:Capacitor
- added D1: Diode, POWER_DIODE_SMD:TO-277A, symbol Power_diode:Diode
- added D2: LED, GENERAL_2-PIN_PLASTIC_SMD:LED0603(1608M), symbol Basic_passive_components:LED
- added H1, H2: MountingHole, MOUNTINGHOLE:MountingHole, symbol MountingHole:MountingHole
- added J1: Conn_02x02, CONNECTOR:Conn-02x02, symbol Link_W2B_connector:Conn_02x02
- added Q1, Q2: CSD18540Q5B, POWER_TRANSISTOR_SMD:SON-8_5x6_M, symbol Power_transistor:CSD18540Q5B
- added Q3: 8050, GENERAL_SMALL-SEMI_SMD:SOT-23, symbol Basic_semiconductor:BJT_NPN
- added R1: 9K, GENERAL_RCL_SMD:R0402(1005M), symbol Basic_passive_components:Resistor
- added R10, R11, R8: 10K, GENERAL_RCL_SMD:R0402(1005M), symbol Basic_passive_components:Resistor
- added R2, R9: 100, GENERAL_RCL_SMD:R0402(1005M), symbol Basic_passive_components:Resistor
- added R3: 200K, GENERAL_RCL_SMD:R0402(1005M), symbol Basic_passive_components:Resistor
- added R4: 100K, GENERAL_RCL_SMD:R0402(1005M), symbol Basic_passive_components:Resistor
- added R5: 38.3K, GENERAL_RCL_SMD:R0402(1005M), symbol Basic_passive_components:Resistor
- added R6: 14K, GENERAL_RCL_SMD:R0402(1005M), symbol Basic_passive_components:Resistor
- added R7: 47K, GENERAL_RCL_SMD:R0402(1005M), symbol Basic_passive_components:Resistor
- added U1: LM5060, GENERAL_MIDDLE-SEMI_SMD:MSOP-3030_10, symbol Integrated-circuit_transistor_driver:LM5060
- added U2: LM5050-1, GENERAL_SMALL-SEMI_SMD:SOT-23-6, symbol Integrated-circuit_transistor_driver:LM5050-1
Connections:
- net EN: now also Q3.3 (Collector), R7.1, R8.1, U1.5 (EN)
- net GND: now also C1.2, C3.1, C4.1, D2.K, J1.1, J1.2, J1.4, Q3.2 (Emitter), R10.1, R6.1, R8.2, U1.6 (GND), U2.2 (GND), U2.3 (OFF)
- net NMOS_IN: now also C1.1, H1., Q2.D (Drain), R1.1, R3.2, R4.1, R7.2, U1.2 (Vin)
- net NMOS_OUT: now also D1.K (Cathode), H2., Q1.D (Drain), R2.2, U2.6 (OUT)
- net ~{EN}: now also J1.3, R9.1
- new net: D1.A (Anode), Q1.S (Source)
- new net: R2.1, U2.1 (VS)
- new net: Q2.S (Source), R11.2, U1.9 (OUT), U2.4 (IN)
- new net: Q1.G (Gate), U2.5 (GATE)
- new net: R4.2, U1.8 (nPGD)
- new net: C4.2, Q3.1 (Base), R10.2, R9.2
- new net: R1.2, U1.1 (SENSE)
- new net: Q2.G (Gate), U1.10 (GATE)
- new net: R5.2, R6.2, U1.3 (OVP)
- new net: R3.1, R5.1, U1.4 (UVLO)
- new net: C3.2, U1.7 (TIMER)
- new net: D2.A, R11.1

Commit message: final
Parts:
- removed D2: LED, GENERAL_2-PIN_PLASTIC_SMD:LED0603(1608M), symbol Basic_passive_components:LED
- added D2: Diode_LED, GENERAL_2-PIN_PLASTIC_SMD:LED0603(1608M), symbol Basic_semiconductor:Diode_LED
- Q1, Q2: footprint POWER_TRANSISTOR_SMD:SON-8_5x6_M -> POWER_TRANSISTOR_SMD:SON-6050-FET
Connections:
- net GND: now also D2.1 (Cathode)
- net NMOS_IN: now also H1.1; no longer H1.
- net NMOS_OUT: now also H2.1; no longer H2.
- net at R11.1: now also D2.2 (Anode)
Changed lines of the file:
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@@
     (stroke (width 0) (type default) (color 0 0 0 0))
   )
-  (wire (pts (xy 163.83 93.98) (xy 163.83 95.25))
+  (wire (pts (xy 163.83 93.98) (xy 163.83 96.52))
     (stroke (width 0) (type default) (color 0 0 0 0))
   )
@@
     (stroke (width 0) (type default) (color 0 0 0 0))
   )
-  (wire (pts (xy 163.83 105.41) (xy 163.83 109.22))
+  (wire (pts (xy 163.83 106.68) (xy 163.83 109.22))
     (stroke (width 0) (type default) (color 0 0 0 0))
   )
@@
   (label "NMOS_OUT" (at 220.98 44.45 0)
     (effects (font (size 1.27 1.27)) (justify left bottom))
-  )
-  (symbol (lib_id "MountingHole:MountingHole") (at 203.2 41.91 0) (unit 1)
-    (in_bom yes) (on_board yes) (fields_autoplaced)
-    (property "Reference" "H1" (id 0) (at 205.605 48.1984 0)
-      (effects (font (size 1.27 1.27)) (justify left))
-    )
-    (property "Value" "MountingHole" (id 1) (at 205.605 50.9735 0)
-      (effects (font (size 1.27 1.27)) (justify left))
-    )
-    (property "Footprint" "MOUNTINGHOLE:MountingHole" (id 2) (at 203.2 41.91 0)
-      (effects (font (size 1.27 1.27)) hide)
-    )
-    (property "Datasheet" "" (id 3) (at 203.2 41.91 0)
-      (effects (font (size 1.27 1.27)) hide)
-    )
-    (pin "")
   )
   (symbol (lib_id "Power_diode:Diode") (at 203.2 72.39 90) (unit 1)
@@
     (pin "1")
     (pin "2")
-  )
-  (symbol (lib_id "MountingHole:MountingHole") (at 220.98 41.91 0) (unit 1)
-    (in_bom yes) (on_board yes) (fields_autoplaced)
-    (property "Reference" "H2" (id 0) (at 223.385 48.1984 0)
-      (effects (font (size 1.27 1.27)) (justify left))
-    )
-    (property "Value" "MountingHole" (id 1) (at 223.385 50.9735 0)
-      (effects (font (size 1.27 1.27)) (justify left))
-    )
-    (property "Footprint" "MOUNTINGHOLE:MountingHole" (id 2) (at 220.98 41.91 0)
-      (effects (font (size 1.27 1.27)) hide)
-    )
-    (property "Datasheet" "" (id 3) (at 220.98 41.91 0)
-      (effects (font (size 1.27 1.27)) hide)
-    )
-    (pin "")
   )
   (symbol (lib_id "Integrated-circuit_transistor_driver:LM5060") (at 125.73 73.66 0) (unit 1)
@@
     (pin "2")
   )
+  (symbol (lib_id "MountingHole:MountingHole") (at 220.98 49.53 0) (unit 1)
+    (in_bom yes) (on_board yes) (fields_autoplaced)
+    (property "Reference" "H2" (id 0) (at 223.385 48.1984 0)
+      (effects (font (size 1.27 1.27)) (justify left))
+    )
+    (property "Value" "MountingHole" (id 1) (at 223.385 50.9735 0)
+      (effects (font (size 1.27 1.27)) (justify left))
+    )
+    (property "Footprint" "MOUNTINGHOLE:MountingHole" (id 2) (at 220.98 49.53 0)
+      (effects (font (size 1.27 1.27)) hide)
+    )
+    (property "Datasheet" "" (id 3) (at 220.98 49.53 0)
+      (effects (font (size 1.27 1.27)) hide)
+    )
+    (pin "1")
+  )
   (symbol (lib_id "Power_transistor:CSD18540Q5B") (at 148.59 73.66 0) (unit 1)
     (in_bom yes) (on_board yes)
@@
       (effects (font (size 1.27 1.27)) (justify left))
     )
-    (property "Footprint" "POWER_TRANSISTOR_SMD:SON-8_5x6_M" (id 2) (at 170.18 69.85 0)
+    (property "Footprint" "POWER_TRANSISTOR_SMD:SON-6050-FET" (id 2) (at 170.18 69.85 0)
       (effects (font (size 1.27 1.27)) hide)
     )
@@
       (effects (font (size 1.27 1.27)) (justify left))
     )
-    (property "Footprint" "POWER_TRANSISTOR_SMD:SON-8_5x6_M" (id 2) (at 212.09 77.47 0)
+    (property "Footprint" "POWER_TRANSISTOR_SMD:SON-6050-FET" (id 2) (at 212.09 77.47 0)
       (effects (font (size 1.27 1.27)) hide)
     )
@@
     (pin "3")
   )
-  (symbol (lib_id "Basic_passive_components:LED") (at 161.29 100.33 90) (unit 1)
-    (in_bom yes) (on_board yes) (fields_autoplaced)
-    (property "Reference" "D2" (id 0) (at 165.735 101.3646 90)
-      (effects (font (size 1.27 1.27)) (justify right))
-    )
-    (property "Value" "LED" (id 1) (at 165.735 104.1397 90)
-      (effects (font (size 1.27 1.27)) (justify right))
-    )
-    (property "Footprint" "GENERAL_2-PIN_PLASTIC_SMD:LED0603(1608M)" (id 2) (at 161.29 100.33 0)
-      (effects (font (size 1.27 1.27)) hide)
-    )
-    (property "Datasheet" "" (id 3) (at 161.29 100.33 0)
-      (effects (font (size 1.27 1.27)) hide)
-    )
-    (pin "A")
-    (pin "K")
-  )
   (symbol (lib_id "Basic_passive_components:Resistor") (at 34.29 85.09 0) (unit 1)
     (in_bom yes) (on_board yes) (fields_autoplaced)
@@
     (pin "1")
   )
+  (symbol (lib_id "Basic_semiconductor:Diode_LED") (at 163.83 101.6 90) (unit 1)
+    (in_bom yes) (on_board yes) (fields_autoplaced)
+    (property "Reference" "D2" (id 0) (at 167.0812 100.6915 90)
+      (effects (font (size 1.27 1.27)) (justify right))
+    )
+    (property "Value" "Diode_LED" (id 1) (at 167.0812 103.4666 90)
+      (effects (font (size 1.27 1.27)) (justify right))
+    )
+    (property "Footprint" "GENERAL_2-PIN_PLASTIC_SMD:LED0603(1608M)" (id 2) (at 163.83 101.6 0)
+      (effects (font (size 1.27 1.27)) hide)
+    )
+    (property "Datasheet" "" (id 3) (at 163.83 101.6 0)
+      (effects (font (size 1.27 1.27)) hide)
+    )
+    (pin "1")
+    (pin "2")
+  )
   (symbol (lib_id "power:GND") (at 100.33 91.44 0) (unit 1)
     (in_bom yes) (on_board yes) (fields_autoplaced)
@@
     )
     (property "Datasheet" "~" (id 3) (at 37.084 134.112 0)
+      (effects (font (size 1.27 1.27)) hide)
+    )
+    (pin "1")
+  )
+  (symbol (lib_id "MountingHole:MountingHole") (at 203.2 49.53 0) (unit 1)
+    (in_bom yes) (on_board yes) (fields_autoplaced)
+    (property "Reference" "H1" (id 0) (at 205.605 48.1984 0)
+      (effects (font (size 1.27 1.27)) (justify left))
+    )
+    (property "Value" "MountingHole" (id 1) (at 205.605 50.9735 0)
+      (effects (font (size 1.27 1.27)) (justify left))
+    )
+    (property "Footprint" "MOUNTINGHOLE:MountingHole" (id 2) (at 203.2 49.53 0)
+      (effects (font (size 1.27 1.27)) hide)
+    )
+    (property "Datasheet" "" (id 3) (at 203.2 49.53 0)
       (effects (font (size 1.27 1.27)) hide)
     )
@@
       (reference "D1") (unit 1) (value "Diode") (footprint "POWER_DIODE_SMD:TO-277A")
     )
-    (path "/bdba0e08-f386-439b-b9d1-35b4ce016bd8"
-      (reference "D2") (unit 1) (value "LED") (footprint "GENERAL_2-PIN_PLASTIC_SMD:LED0603(1608M)")
-    )
-    (path "/02be2094-fd60-4d2f-9ad9-43f982c1e650"
+    (path "/c839b541-5f15-4bff-8881-7c03afd82c4e"
+      (reference "D2") (unit 1) (value "Diode_LED") (footprint "GENERAL_2-PIN_PLASTIC_SMD:LED0603(1608M)")
+    )
+    (path "/cfd2b6bc-75a2-4187-872c-2427d5d3cad3"
       (reference "H1") (unit 1) (value "MountingHole") (footprint "MOUNTINGHOLE:MountingHole")
     )
-    (path "/3b9b8270-8548-4508-97fd-ea0028a8c5e3"
+    (path "/545caeb8-9f21-4b24-ab9f-1f30004c26af"
       (reference "H2") (unit 1) (value "MountingHole") (footprint "MOUNTINGHOLE:MountingHole")
     )
@@
     )
     (path "/ae8a643e-c295-4bca-8057-36d6e8cf2a88"
-      (reference "Q1") (unit 1) (value "CSD18540Q5B") (footprint "POWER_TRANSISTOR_SMD:SON-8_5x6_M")
+      (reference "Q1") (unit 1) (value "CSD18540Q5B") (footprint "POWER_TRANSISTOR_SMD:SON-6050-FET")
     )
     (path "/55aec6e8-9443-4619-9906-18423b70dd76"
-      (reference "Q2") (unit 1) (value "CSD18540Q5B") (footprint "POWER_TRANSISTOR_SMD:SON-8_5x6_M")
+      (reference "Q2") (unit 1) (value "CSD18540Q5B") (footprint "POWER_TRANSISTOR_SMD:SON-6050-FET")
     )
     (path "/bc2effa5-92d1-4065-b9cf-ed76ac660f73"

Commit message: GERBER project
Parts:
- C3, C4: footprint GENERAL_RCL_SMD:C0402(1005M) -> GENERAL_RCL_SMD:C0603(1608M)
- H1, H2: footprint MOUNTINGHOLE:MountingHole -> MountingHole:mountinghole
- J1: footprint CONNECTOR:Conn-02x02 -> CONNECTOR_Odd_Even:Conn_02x02
- R10, R11, R2, R3, R4, R5, R6, R8, R9: footprint GENERAL_RCL_SMD:R0402(1005M) -> GENERAL_RCL_SMD:R0603(1608M)
Changed lines of the file:
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@@
       (effects (font (size 1.27 1.27)) (justify left))
     )
-    (property "Footprint" "GENERAL_RCL_SMD:R0402(1005M)" (id 2) (at 139.7 55.88 0)
+    (property "Footprint" "GENERAL_RCL_SMD:R0603(1608M)" (id 2) (at 139.7 55.88 0)
       (effects (font (size 1.27 1.27)) hide)
     )
@@
       (effects (font (size 1.27 1.27)) (justify right))
     )
-    (property "Footprint" "GENERAL_RCL_SMD:C0402(1005M)" (id 2) (at 41.91 92.71 0)
+    (property "Footprint" "GENERAL_RCL_SMD:C0603(1608M)" (id 2) (at 41.91 92.71 0)
       (effects (font (size 1.27 1.27)) hide)
     )
@@
     (property "Reference" "R5" (id 0) (at 105.41 68.5505 0))
     (property "Value" "38.3K" (id 1) (at 105.41 71.3256 0))
-    (property "Footprint" "GENERAL_RCL_SMD:R0402(1005M)" (id 2) (at 109.22 77.47 0)
+    (property "Footprint" "GENERAL_RCL_SMD:R0603(1608M)" (id 2) (at 109.22 77.47 0)
       (effects (font (size 1.27 1.27)) hide)
     )
@@
       (effects (font (size 1.27 1.27)) (justify left))
     )
-    (property "Footprint" "MOUNTINGHOLE:MountingHole" (id 2) (at 220.98 49.53 0)
+    (property "Footprint" "MountingHole:mountinghole" (id 2) (at 220.98 49.53 0)
       (effects (font (size 1.27 1.27)) hide)
     )
@@
       (effects (font (size 1.27 1.27)) (justify right))
     )
-    (property "Footprint" "GENERAL_RCL_SMD:C0402(1005M)" (id 2) (at 138.43 86.36 0)
+    (property "Footprint" "GENERAL_RCL_SMD:C0603(1608M)" (id 2) (at 138.43 86.36 0)
       (effects (font (size 1.27 1.27)) hide)
     )
@@
       (effects (font (size 1.27 1.27)) (justify left))
     )
-    (property "Footprint" "GENERAL_RCL_SMD:R0402(1005M)" (id 2) (at 72.39 77.47 0)
+    (property "Footprint" "GENERAL_RCL_SMD:R0603(1608M)" (id 2) (at 72.39 77.47 0)
       (effects (font (size 1.27 1.27)) hide)
     )
@@
       (effects (font (size 1.27 1.27)) (justify right))
     )
-    (property "Footprint" "GENERAL_RCL_SMD:R0402(1005M)" (id 2) (at 96.52 87.63 0)
+    (property "Footprint" "GENERAL_RCL_SMD:R0603(1608M)" (id 2) (at 96.52 87.63 0)
       (effects (font (size 1.27 1.27)) hide)
     )
@@
       (effects (font (size 1.27 1.27)) (justify right))
     )
-    (property "Footprint" "GENERAL_RCL_SMD:R0402(1005M)" (id 2) (at 160.02 92.71 0)
+    (property "Footprint" "GENERAL_RCL_SMD:R0603(1608M)" (id 2) (at 160.02 92.71 0)
       (effects (font (size 1.27 1.27)) hide)
     )
@@
     (property "Reference" "R2" (id 0) (at 195.6095 88.9 0))
     (property "Value" "100" (id 1) (at 192.8344 88.9 0))
-    (property "Footprint" "GENERAL_RCL_SMD:R0402(1005M)" (id 2) (at 186.69 92.71 0)
+    (property "Footprint" "GENERAL_RCL_SMD:R0603(1608M)" (id 2) (at 186.69 92.71 0)
       (effects (font (size 1.27 1.27)) hide)
     )
@@
     (property "Reference" "R9" (id 0) (at 34.29 79.9805 0))
     (property "Value" "100" (id 1) (at 34.29 82.7556 0))
-    (property "Footprint" "GENERAL_RCL_SMD:R0402(1005M)" (id 2) (at 30.48 81.28 0)
+    (property "Footprint" "GENERAL_RCL_SMD:R0603(1608M)" (id 2) (at 30.48 81.28 0)
       (effects (font (size 1.27 1.27)) hide)
     )
@@
       (effects (font (size 1.27 1.27)) (justify left))
     )
-    (property "Footprint" "MOUNTINGHOLE:MountingHole" (id 2) (at 203.2 49.53 0)
+    (property "Footprint" "MountingHole:mountinghole" (id 2) (at 203.2 49.53 0)
       (effects (font (size 1.27 1.27)) hide)
     )
@@
       (effects (font (size 1.27 1.27)) (justify right))
     )
-    (property "Footprint" "GENERAL_RCL_SMD:R0402(1005M)" (id 2) (at 106.68 67.31 0)
+    (property "Footprint" "GENERAL_RCL_SMD:R0603(1608M)" (id 2) (at 106.68 67.31 0)
       (effects (font (size 1.27 1.27)) hide)
     )
@@
       (effects (font (size 1.27 1.27)) hide)
     )
-    (property "Footprint" "CONNECTOR:Conn-02x02" (id 2) (at 119.38 27.94 0)
+    (property "Footprint" "CONNECTOR_Odd_Even:Conn_02x02" (id 2) (at 119.38 27.94 0)
       (effects (font (size 1.27 1.27)) hide)
     )
@@
       (effects (font (size 1.27 1.27)) (justify right))
     )
-    (property "Footprint" "GENERAL_RCL_SMD:R0402(1005M)" (id 2) (at 43.18 96.52 0)
+    (property "Footprint" "GENERAL_RCL_SMD:R0603(1608M)" (id 2) (at 43.18 96.52 0)
       (effects (font (size 1.27 1.27)) hide)
     )
@@
     )
     (path "/77c4a6d8-a2d2-461d-b88b-00a8e5d84abc"
-      (reference "C3") (unit 1) (value "100n") (footprint "GENERAL_RCL_SMD:C0402(1005M)")
+      (reference "C3") (unit 1) (value "100n") (footprint "GENERAL_RCL_SMD:C0603(1608M)")
     )
     (path "/201c9bac-f9c3-418c-9c8e-2fc92c88c82a"
-      (reference "C4") (unit 1) (value "100n") (footprint "GENERAL_RCL_SMD:C0402(1005M)")
+      (reference "C4") (unit 1) (value "100n") (footprint "GENERAL_RCL_SMD:C0603(1608M)")
     )
     (path "/06d72d7f-a993-46d9-aa59-e05517035829"
@@
     )
     (path "/cfd2b6bc-75a2-4187-872c-2427d5d3cad3"
-      (reference "H1") (unit 1) (value "MountingHole") (footprint "MOUNTINGHOLE:MountingHole")
+      (reference "H1") (unit 1) (value "MountingHole") (footprint "MountingHole:mountinghole")
     )
     (path "/545caeb8-9f21-4b24-ab9f-1f30004c26af"
-      (reference "H2") (unit 1) (value "MountingHole") (footprint "MOUNTINGHOLE:MountingHole")
+      (reference "H2") (unit 1) (value "MountingHole") (footprint "MountingHole:mountinghole")
     )
     (path "/e0af243e-0a28-464d-abd0-34b7d09bfc35"
-      (reference "J1") (unit 1) (value "Conn_02x02") (footprint "CONNECTOR:Conn-02x02")
+      (reference "J1") (unit 1) (value "Conn_02x02") (footprint "CONNECTOR_Odd_Even:Conn_02x02")
     )
     (path "/ae8a643e-c295-4bca-8057-36d6e8cf2a88"
@@
     )
     (path "/bb6b5f44-6816-4efe-a63a-da7a86ea7699"
-      (reference "R2") (unit 1) (value "100") (footprint "GENERAL_RCL_SMD:R0402(1005M)")
+      (reference "R2") (unit 1) (value "100") (footprint "GENERAL_RCL_SMD:R0603(1608M)")
     )
     (path "/d0ab4222-20e2-4cec-a167-3ce49c815802"
-      (reference "R3") (unit 1) (value "200K") (footprint "GENERAL_RCL_SMD:R0402(1005M)")
+      (reference "R3") (unit 1) (value "200K") (footprint "GENERAL_RCL_SMD:R0603(1608M)")
     )
     (path "/15382cd3-640b-47a2-926f-51136398a448"
-      (reference "R4") (unit 1) (value "100K") (footprint "GENERAL_RCL_SMD:R0402(1005M)")
+      (reference "R4") (unit 1) (value "100K") (footprint "GENERAL_RCL_SMD:R0603(1608M)")
     )
     (path "/4a6ada35-c9f8-4543-942e-44f4a8e7133b"
-      (reference "R5") (unit 1) (value "38.3K") (footprint "GENERAL_RCL_SMD:R0402(1005M)")
+      (reference "R5") (unit 1) (value "38.3K") (footprint "GENERAL_RCL_SMD:R0603(1608M)")
     )
     (path "/7d96d093-c667-4b56-bd73-cc24d39bfa58"
-      (reference "R6") (unit 1) (value "14K") (footprint "GENERAL_RCL_SMD:R0402(1005M)")
+      (reference "R6") (unit 1) (value "14K") (footprint "GENERAL_RCL_SMD:R0603(1608M)")
     )
     (path "/7cc752c2-5a6c-41b2-92ba-3951097cdd2b"
@@
     )
     (path "/7d0b73c4-ecc7-4362-9ae1-df1ea1d895ac"
-      (reference "R8") (unit 1) (value "10K") (footprint "GENERAL_RCL_SMD:R0402(1005M)")
+      (reference "R8") (unit 1) (value "10K") (footprint "GENERAL_RCL_SMD:R0603(1608M)")
     )
     (path "/be1738ee-f11f-4664-aff1-46e6f8fa0cb0"
-      (reference "R9") (unit 1) (value "100") (footprint "GENERAL_RCL_SMD:R0402(1005M)")
+      (reference "R9") (unit 1) (value "100") (footprint "GENERAL_RCL_SMD:R0603(1608M)")
     )
     (path "/e23ab1ee-3deb-450d-aed8-90c316fd97ba"
-      (reference "R10") (unit 1) (value "10K") (footprint "GENERAL_RCL_SMD:R0402(1005M)")
+      (reference "R10") (unit 1) (value "10K") (footprint "GENERAL_RCL_SMD:R0603(1608M)")
     )
     (path "/b04a0007-7c3f-4651-bf02-4215a692858e"
-      (reference "R11") (unit 1) (value "10K") (footprint "GENERAL_RCL_SMD:R0402(1005M)")
+      (reference "R11") (unit 1) (value "10K") (footprint "GENERAL_RCL_SMD:R0603(1608M)")
     )
     (path "/3c931f9d-b05a-4411-a471-b9d1498920ed"

Commit message: another right version
Connections:
- net at D1.A (Anode), Q1.S (Source): now also Q2.S (Source), R11.2, U1.9 (OUT), U2.4 (IN)
Changed lines of the file:
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@@
   (junction (at 163.83 78.74) (diameter 0) (color 0 0 0 0)
+  )
+  (junction (at 190.5 66.04) (diameter 0) (color 0 0 0 0)
   )
   (junction (at 119.38 53.34) (diameter 0) (color 0 0 0 0)
@@
     (stroke (width 0) (type default) (color 0 0 0 0))
   )
+  (wire (pts (xy 163.83 66.04) (xy 190.5 66.04))
+    (stroke (width 0) (type default) (color 0 0 0 0))
+  )
   (wire (pts (xy 163.83 83.82) (xy 163.83 78.74))
     (stroke (width 0) (type default) (color 0 0 0 0))
@@
     (stroke (width 0) (type default) (color 0 0 0 0))
   )
+  (wire (pts (xy 163.83 78.74) (xy 163.83 66.04))
+    (stroke (width 0) (type default) (color 0 0 0 0))
+  )
