File: HighSideSwitch.kicad_sch (KiCad schematic)
At the start: 21 parts, among them J1 Conn_02x02_Odd_Even, Q1 CSD18540Q5B, Q2 CSD18540Q5B, Q3 Q_Dual_NPN_NPN_E1B1C2E2B2C1, U1 LM5060

Commit message: Update LM5060
Parts:
- R3: value 60k -> 10k
- R6: value 4.7k -> 10k
Connections:
- net GND: no longer D2.1 (K)
- net at R6.2, U1.3 (OVP): no longer R3.2, U1.4 (UVLO)
- net PGD: now reaches U1.8 (~{PGD})
- net PGD: now also D2.1 (K)
- new net: R3.2, U1.4 (UVLO)
- no-connect marks 1 -> 0
Other:
- moved on the sheet: D2, R11, R5
Changed lines of the file:
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@@
   (junction (at 154.94 51.435) (diameter 0) (color 0 0 0 0)
   )
-  (junction (at 96.52 83.82) (diameter 0) (color 0 0 0 0)
-  )
   (junction (at 83.82 51.435) (diameter 0) (color 0 0 0 0)
   )
@@
   (junction (at 76.2 83.82) (diameter 0) (color 0 0 0 0)
   )
-  (junction (at 161.29 51.435) (diameter 0) (color 0 0 0 0)
-  )
   (junction (at 147.32 60.325) (diameter 0) (color 0 0 0 0)
   )
   (junction (at 83.82 75.565) (diameter 0) (color 0 0 0 0)
   )
-  (junction (at 96.52 81.28) (diameter 0) (color 0 0 0 0)
-  )
   (junction (at 130.81 51.435) (diameter 0) (color 0 0 0 0)
   )
+  (junction (at 161.925 51.435) (diameter 0) (color 0 0 0 0)
+  )
   (junction (at 106.68 51.435) (diameter 0) (color 0 0 0 0)
   )
@@
   (junction (at 83.82 93.98) (diameter 0) (color 0 0 0 0)
   )
-  (no_connect (at 121.92 83.82))
   (wire (pts (xy 116.205 60.325) (xy 114.3 60.325))
     (stroke (width 0) (type default) (color 0 0 0 0))
@@
     (stroke (width 0) (type default) (color 0 0 0 0))
   )
-  (wire (pts (xy 161.29 51.435) (xy 167.005 51.435))
-    (stroke (width 0) (type default) (color 0 0 0 0))
-  )
   (wire (pts (xy 101.6 83.82) (xy 96.52 83.82))
     (stroke (width 0) (type default) (color 0 0 0 0))
@@
     (stroke (width 0) (type default) (color 0 0 0 0))
   )
-  (wire (pts (xy 154.94 51.435) (xy 161.29 51.435))
-    (stroke (width 0) (type default) (color 0 0 0 0))
-  )
-  (wire (pts (xy 140.97 81.28) (xy 140.97 84.455))
+  (wire (pts (xy 154.94 51.435) (xy 161.925 51.435))
+    (stroke (width 0) (type default) (color 0 0 0 0))
+  )
+  (wire (pts (xy 140.97 81.28) (xy 140.97 87.63))
     (stroke (width 0) (type default) (color 0 0 0 0))
   )
@@
     (stroke (width 0) (type default) (color 0 0 0 0))
   )
-  (wire (pts (xy 161.29 68.58) (xy 161.29 80.01))
+  (wire (pts (xy 161.925 62.865) (xy 161.925 72.39))
     (stroke (width 0) (type default) (color 0 0 0 0))
   )
@@
     (stroke (width 0) (type default) (color 0 0 0 0))
   )
+  (wire (pts (xy 161.925 51.435) (xy 167.005 51.435))
+    (stroke (width 0) (type default) (color 0 0 0 0))
+  )
   (wire (pts (xy 123.825 63.5) (xy 123.825 60.325))
     (stroke (width 0) (type default) (color 0 0 0 0))
@@
     (stroke (width 0) (type default) (color 0 0 0 0))
   )
+  (wire (pts (xy 161.925 51.435) (xy 161.925 57.785))
+    (stroke (width 0) (type default) (color 0 0 0 0))
+  )
   (wire (pts (xy 54.61 43.815) (xy 55.88 43.815))
     (stroke (width 0) (type default) (color 0 0 0 0))
@@
     (stroke (width 0) (type default) (color 0 0 0 0))
   )
-  (wire (pts (xy 161.29 87.63) (xy 161.29 93.98))
-    (stroke (width 0) (type default) (color 0 0 0 0))
-  )
   (wire (pts (xy 83.82 51.435) (xy 96.52 51.435))
     (stroke (width 0) (type default) (color 0 0 0 0))
@@
     (stroke (width 0) (type default) (color 0 0 0 0))
   )
-  (wire (pts (xy 140.97 89.535) (xy 140.97 93.345))
+  (wire (pts (xy 140.97 92.71) (xy 140.97 93.345))
     (stroke (width 0) (type default) (color 0 0 0 0))
   )
@@
     (stroke (width 0) (type default) (color 0 0 0 0))
   )
-  (wire (pts (xy 96.52 81.28) (xy 96.52 83.82))
-    (stroke (width 0) (type default) (color 0 0 0 0))
-  )
   (wire (pts (xy 130.81 51.435) (xy 130.81 71.755))
     (stroke (width 0) (type default) (color 0 0 0 0))
@@
     (stroke (width 0) (type default) (color 0 0 0 0))
   )
-  (wire (pts (xy 161.29 51.435) (xy 161.29 63.5))
-    (stroke (width 0) (type default) (color 0 0 0 0))
-  )
   (wire (pts (xy 121.92 81.28) (xy 127.635 81.28))
     (stroke (width 0) (type default) (color 0 0 0 0))
@@
   )
   (wire (pts (xy 64.135 83.82) (xy 67.31 83.82))
+    (stroke (width 0) (type default) (color 0 0 0 0))
+  )
+  (wire (pts (xy 161.925 80.01) (xy 161.925 93.345))
     (stroke (width 0) (type default) (color 0 0 0 0))
   )
@@
     (effects (font (size 1.27 1.27)) (justify right bottom))
   )
+  (label "PGD" (at 161.925 93.345 0)
+    (effects (font (size 1.27 1.27)) (justify left bottom))
+  )
   (label "NMOS_OUT" (at 167.005 51.435 0)
+    (effects (font (size 1.27 1.27)) (justify left bottom))
+  )
+  (label "PGD" (at 121.92 83.82 0)
     (effects (font (size 1.27 1.27)) (justify left bottom))
   )
@@
     (pin "2")
   )
-  (symbol (lib_id "power:GND") (at 161.29 93.98 0) (mirror y) (unit 1)
-    (in_bom yes) (on_board yes) (fields_autoplaced)
-    (property "Reference" "#PWR010" (id 0) (at 161.29 100.33 0)
-      (effects (font (size 1.27 1.27)) hide)
-    )
-    (property "Value" "GND" (id 1) (at 163.195 95.6838 0)
-      (effects (font (size 1.27 1.27)) (justify right))
-    )
-    (property "Footprint" "" (id 2) (at 161.29 93.98 0)
-      (effects (font (size 1.27 1.27)) hide)
-    )
-    (property "Datasheet" "" (id 3) (at 161.29 93.98 0)
-      (effects (font (size 1.27 1.27)) hide)
-    )
-    (pin "1")
-  )
   (symbol (lib_id "Mechanical:MountingHole_Pad") (at 191.135 48.26 180) (unit 1)
     (in_bom yes) (on_board yes) (fields_autoplaced)
@@
     (pin "2")
   )
-  (symbol (lib_id "Device:LED") (at 161.29 83.82 90) (unit 1)
-    (in_bom yes) (on_board yes)
-    (property "Reference" "D2" (id 0) (at 162.814 80.264 90)
-      (effects (font (size 1.27 1.27)) (justify right))
-    )
-    (property "Value" "LED" (id 1) (at 162.56 90.424 90)
-      (effects (font (size 1.27 1.27)) (justify right))
-    )
-    (property "Footprint" "LED_SMD:LED_0603_1608Metric" (id 2) (at 161.29 83.82 0)
-      (effects (font (size 1.27 1.27)) hide)
-    )
-    (property "Datasheet" "~" (id 3) (at 161.29 83.82 0)
+  (symbol (lib_id "Device:LED") (at 161.925 76.2 90) (unit 1)
+    (in_bom yes) (on_board yes)
+    (property "Reference" "D2" (id 0) (at 163.449 72.644 90)
+      (effects (font (size 1.27 1.27)) (justify right))
+    )
+    (property "Value" "LED" (id 1) (at 163.195 82.804 90)
+      (effects (font (size 1.27 1.27)) (justify right))
+    )
+    (property "Footprint" "LED_SMD:LED_0603_1608Metric" (id 2) (at 161.925 76.2 0)
+      (effects (font (size 1.27 1.27)) hide)
+    )
+    (property "Datasheet" "~" (id 3) (at 161.925 76.2 0)
       (effects (font (size 1.27 1.27)) hide)
     )
@@
       (effects (font (size 1.27 1.27)) (justify left))
     )
-    (property "Value" "60k" (id 1) (at 96.52 71.501 0)
+    (property "Value" "10k" (id 1) (at 96.52 71.501 0)
       (effects (font (size 1.27 1.27)) (justify left))
     )
@@
       (effects (font (size 1.27 1.27)) (justify right))
     )
-    (property "Value" "4.7k" (id 1) (at 91.694 91.821 0)
+    (property "Value" "10k" (id 1) (at 91.694 91.821 0)
       (effects (font (size 1.27 1.27)) (justify right))
     )
@@
     (pin "1")
   )
-  (symbol (lib_id "Device:R_Small") (at 140.97 86.995 0) (unit 1)
-    (in_bom yes) (on_board yes)
-    (property "Reference" "R5" (id 0) (at 138.684 84.201 0)
-      (effects (font (size 1.27 1.27)) (justify left))
-    )
-    (property "Value" "10k" (id 1) (at 140.97 90.551 0)
-      (effects (font (size 1.27 1.27)) (justify left))
-    )
-    (property "Footprint" "Resistor_SMD:R_0402_1005Metric" (id 2) (at 140.97 86.995 0)
-      (effects (font (size 1.27 1.27)) hide)
-    )
-    (property "Datasheet" "~" (id 3) (at 140.97 86.995 0)
+  (symbol (lib_id "Device:R_Small") (at 140.97 90.17 0) (unit 1)
+    (in_bom yes) (on_board yes)
+    (property "Reference" "R5" (id 0) (at 138.684 87.376 0)
+      (effects (font (size 1.27 1.27)) (justify left))
+    )
+    (property "Value" "10k" (id 1) (at 140.97 93.726 0)
+      (effects (font (size 1.27 1.27)) (justify left))
+    )
+    (property "Footprint" "Resistor_SMD:R_0402_1005Metric" (id 2) (at 140.97 90.17 0)
+      (effects (font (size 1.27 1.27)) hide)
+    )
+    (property "Datasheet" "~" (id 3) (at 140.97 90.17 0)
       (effects (font (size 1.27 1.27)) hide)
     )
@@
     (pin "2")
   )
-  (symbol (lib_id "Device:R_Small") (at 161.29 66.04 0) (unit 1)
-    (in_bom yes) (on_board yes)
-    (property "Reference" "R11" (id 0) (at 161.29 62.865 0)
-      (effects (font (size 1.27 1.27)) (justify left))
-    )
-    (property "Value" "10K" (id 1) (at 161.29 69.596 0)
-      (effects (font (size 1.27 1.27)) (justify left))
-    )
-    (property "Footprint" "Resistor_SMD:R_0402_1005Metric" (id 2) (at 161.29 66.04 0)
-      (effects (font (size 1.27 1.27)) hide)
-    )
-    (property "Datasheet" "~" (id 3) (at 161.29 66.04 0)
+  (symbol (lib_id "Device:R_Small") (at 161.925 60.325 0) (unit 1)
+    (in_bom yes) (on_board yes)
+    (property "Reference" "R11" (id 0) (at 161.925 57.15 0)
+      (effects (font (size 1.27 1.27)) (justify left))
+    )
+    (property "Value" "10K" (id 1) (at 161.925 63.881 0)
+      (effects (font (size 1.27 1.27)) (justify left))
+    )
+    (property "Footprint" "Resistor_SMD:R_0402_1005Metric" (id 2) (at 161.925 60.325 0)
+      (effects (font (size 1.27 1.27)) hide)
+    )
+    (property "Datasheet" "~" (id 3) (at 161.925 60.325 0)
       (effects (font (size 1.27 1.27)) hide)
     )
@@
       (reference "#PWR08") (unit 1) (value "GND") (footprint "")
     )
-    (path "/242a5dcf-04bb-4399-9d12-fb13f6a7c0d6"
-      (reference "#PWR010") (unit 1) (value "GND") (footprint "")
-    )
     (path "/a8b5f16e-c6df-41f9-9209-427d423ec621"
       (reference "#PWR011") (unit 1) (value "GND") (footprint "")
@@
     )
     (path "/5ca6599d-f880-4e04-9824-f166e17b980e"
-      (reference "R3") (unit 1) (value "60k") (footprint "Resistor_SMD:R_0402_1005Metric")
+      (reference "R3") (unit 1) (value "10k") (footprint "Resistor_SMD:R_0402_1005Metric")
     )
     (path "/960d81bb-da7f-4a13-95e5-4c81c539359a"
@@
     )
     (path "/a55aba56-89d8-4475-8c5b-50bf759260e9"
-      (reference "R6") (unit 1) (value "4.7k") (footprint "Resistor_SMD:R_0402_1005Metric")
+      (reference "R6") (unit 1) (value "10k") (footprint "Resistor_SMD:R_0402_1005Metric")
     )
     (path "/5b392dfa-317a-410a-b6f4-469ccf8cb638"
